Commit message: ytoubleshooting for loading the model in gazebo

File: src/amr_project/robot_description/urdf/bot.urdf (robot description, URDF)
Before this commit: robot bot, 6 links, 5 joints
Links:
- link base_link: geometry collision mesh filename=package://amr_project/meshes/base_link.STL; visual mesh filename=package://amr_project/meshes/base_link.STL
- link caster_front_link: geometry collision mesh filename=package://amr_project/meshes/caster_front_link.STL; visual mesh filename=package://amr_project/meshes/caster_front_link.STL
- link caster_rear_link: geometry collision mesh filename=package://amr_project/meshes/caster_rear_link.STL; visual mesh filename=package://amr_project/meshes/caster_rear_link.STL
- link left_wheel_link: geometry collision mesh filename=package://amr_project/meshes/wheel_left_link.STL; visual mesh filename=package://amr_project/meshes/wheel_left_link.STL
- link right_wheel_link: geometry collision mesh filename=package://amr_project/meshes/wheel_right_link.STL; visual mesh filename=package://amr_project/meshes/wheel_right_link.STL
