Commit message: updated the gazebo urdf file for stereo camera setup

File: src/amr_project/robot_description/urdf/bot_gazebo.xacro (robot description, xacro)
@@ -9,9 +9,5 @@
         <maxVel>1.0</maxVel>
         <fdir1>1 0 0</fdir1>
-        <material>
-            <ambient>0.2 0.2 0.2 1</ambient>
-            <diffuse>0.2 0.2 0.2 1</diffuse>
-            <specular>0.1 0.1 0.1 1</specular>
-        </material>
+        <material>Gazebo/Black</material>
     </gazebo>
     <gazebo reference="left_wheel_link">
@@ -23,52 +19,31 @@
         <maxVel>1.0</maxVel>
         <fdir1>1 0 0</fdir1>
-        <material>
-            <ambient>0.2 0.2 0.2 1</ambient>
-            <diffuse>0.2 0.2 0.2 1</diffuse>
-            <specular>0.1 0.1 0.1 1</specular>
-        </material>
+        <material>Gazebo/Black</material>
     </gazebo>
     <gazebo reference="caster_front_link">
-        <mu1>0.01</mu1>
-        <mu2>0.01</mu2>
+        <mu1>0.0</mu1>
+        <mu2>0.0</mu2>
         <kp>1000000.0</kp>
         <kd>100.0</kd>
-        <minDepth>0.001</minDepth>
-        <maxVel>1.0</maxVel>
-        <material>
-            <ambient>0.5 0.5 0.5 1</ambient>
-            <diffuse>0.5 0.5 0.5 1</diffuse>
-        </material>
+        <material>Gazebo/White</material>
     </gazebo>
     <gazebo reference="caster_rear_link">
-        <mu1>0.01</mu1>
-        <mu2>0.01</mu2>
+        <mu1>0.0</mu1>
+        <mu2>0.0</mu2>
         <kp>1000000.0</kp>
         <kd>100.0</kd>
-        <minDepth>0.001</minDepth>
-        <maxVel>1.0</maxVel>
-        <material>
-            <ambient>0.5 0.5 0.5 1</ambient>
-            <diffuse>0.5 0.5 0.5 1</diffuse>
-        </material>
+        <material>Gazebo/White</material>
     </gazebo>
     <gazebo reference="base_link">
-        <material>
-            <ambient>0.0 0.5 1.0 1</ambient>
-            <diffuse>0.0 0.5 1.0 1</diffuse>
-            <specular>0.1 0.1 0.1 1</specular>
-        </material>
+        <material>Gazebo/Blue</material>
     </gazebo>
     <gazebo reference="imu_link">
-        <material>
-            <ambient>1.0 1.0 0.0 1</ambient>
-            <diffuse>1.0 1.0 0.0 1</diffuse>
-        </material>
+        <material>Gazebo/Red</material>
     </gazebo>
     <gazebo reference="laser_link">
-        <material>
-            <ambient>1.0 0.0 1.0 1</ambient>
-            <diffuse>1.0 0.0 1.0 1</diffuse>
-        </material>
+        <material>Gazebo/Red</material>
+    </gazebo>
+    <gazebo reference="camera_mount_link">
+        <material>Gazebo/Black</material>
     </gazebo>
     <gazebo reference="imu_link">
@@ -76,47 +51,16 @@
             <always_on>true</always_on>
             <update_rate>100</update_rate>
-            <visualize>true</visualize>
+            <visualize>false</visualize>
             <topic>imu</topic>
-            <enable_metrics>true</enable_metrics>
             <imu>
                 <angular_velocity>
-                    <x>
-                        <noise type="gaussian">
-                            <mean>0.0</mean>
-                            <stddev>2e-4</stddev>
-                        </noise>
-                    </x>
-                    <y>
-                        <noise type="gaussian">
-                            <mean>0.0</mean>
-                            <stddev>2e-4</stddev>
-                        </noise>
-                    </y>
-                    <z>
-                        <noise type="gaussian">
-                            <mean>0.0</mean>
-                            <stddev>2e-4</stddev>
-                        </noise>
-                    </z>
+                    <x><noise type="gaussian"><mean>0.0</mean><stddev>2e-4</stddev></noise></x>
+                    <y><noise type="gaussian"><mean>0.0</mean><stddev>2e-4</stddev></noise></y>
+                    <z><noise type="gaussian"><mean>0.0</mean><stddev>2e-4</stddev></noise></z>
                 </angular_velocity>
                 <linear_acceleration>
-                    <x>
-                        <noise type="gaussian">
-                            <mean>0.0</mean>
-                            <stddev>1.7e-2</stddev>
-                        </noise>
-                    </x>
-                    <y>
-                        <noise type="gaussian">
-                            <mean>0.0</mean>
-                            <stddev>1.7e-2</stddev>
-                        </noise>
-                    </y>
-                    <z>
-                        <noise type="gaussian">
-                            <mean>0.0</mean>
-                            <stddev>1.7e-2</stddev>
-                        </noise>
-                    </z>
+                    <x><noise type="gaussian"><mean>0.0</mean><stddev>1.7e-2</stddev></noise></x>
+                    <y><noise type="gaussian"><mean>0.0</mean><stddev>1.7e-2</stddev></noise></y>
+                    <z><noise type="gaussian"><mean>0.0</mean><stddev>1.7e-2</stddev></noise></z>
                 </linear_acceleration>
             </imu>
@@ -129,5 +73,4 @@
             <visualize>true</visualize>
             <topic>scan</topic>
-            <enable_metrics>true</enable_metrics>
             <lidar>
                 <scan>
@@ -152,3 +95,78 @@
         </sensor>
     </gazebo>
+    <gazebo reference="camera_left_link">
+        <sensor name="left_camera" type="camera">
+            <always_on>true</always_on>
+            <update_rate>30</update_rate>
+            <visualize>false</visualize>
+            <topic>camera/left</topic>
+            <camera>
+                <horizontal_fov>1.5708</horizontal_fov>
+                <image>
+                    <width>640</width>
+                    <height>480</height>
+                    <format>R8G8B8</format>
+                </image>
+                <clip>
+                    <near>0.05</near>
+                    <far>100</far>
+                </clip>
+                <noise>
+                    <type>gaussian</type>
+                    <mean>0.0</mean>
+                    <stddev>0.007</stddev>
+                </noise>
+            </camera>
+        </sensor>
+    </gazebo>
+    <gazebo reference="camera_right_link">
+        <sensor name="right_camera" type="camera">
+            <always_on>true</always_on>
+            <update_rate>30</update_rate>
+            <visualize>false</visualize>
+            <topic>camera/right</topic>
+            <camera>
+                <horizontal_fov>1.5708</horizontal_fov>
+                <image>
+                    <width>640</width>
+                    <height>480</height>
+                    <format>R8G8B8</format>
+                </image>
+                <clip>
+                    <near>0.05</near>
+                    <far>100</far>
+                </clip>
+                <noise>
+                    <type>gaussian</type>
+                    <mean>0.0</mean>
+                    <stddev>0.007</stddev>
+                </noise>
+            </camera>
+        </sensor>
+    </gazebo>
+    <gazebo reference="camera_center_link">
+        <sensor name="depth_camera" type="depth_camera">
+            <always_on>true</always_on>
+            <update_rate>30</update_rate>
+            <visualize>false</visualize>
+            <topic>camera/depth</topic>
+            <camera>
+                <horizontal_fov>1.5708</horizontal_fov>
+                <image>
+                    <width>640</width>
+                    <height>480</height>
+                    <format>R_FLOAT32</format>
+                </image>
+                <clip>
+                    <near>0.05</near>
+                    <far>10.0</far>
+                </clip>
+                <noise>
+                    <type>gaussian</type>
+                    <mean>0.0</mean>
+                    <stddev>0.01</stddev>
+                </noise>
+            </camera>
+        </sensor>
+    </gazebo>
 </robot>
