Commit message: updated the controller file and gazebo launch file and the setup file

File: src/amr_project/robot_description/urdf/bot.urdf.xacro (robot description, xacro)
@@ -3,5 +3,5 @@
     <xacro:arg name="is_ignition" default="true"/>
     <xacro:include filename="$(find amr_project)/urdf/bot_gazebo.xacro"/>
-    <xacro:include filename="$(find amr_project)/urdf/bot_ros2_control.xacro"/>
+    <xacro:include filename="$(find amr_project)/urdf/amr_controller.xacro"/>
     <link name="base_footprint"/>
     <link name="base_link">
@@ -23,7 +23,7 @@
         <inertial>
             <origin xyz="0 0 0" rpy="0 0 0"/>
-            <mass value="1.0"/>
-            <inertia ixx="0.01" ixy="0.0" ixz="0.0"
-                     iyy="0.01" iyz="0.0" izz="0.01"/>
+            <mass value="5.0"/>
+            <inertia ixx="0.0347" ixy="0.0" ixz="0.0"
+                     iyy="0.0347" iyz="0.0" izz="0.0625"/>
         </inertial>
     </link>
@@ -33,5 +33,5 @@
         <origin xyz="0 0 0.033" rpy="0 0 0"/>
     </joint>
-        <link name="right_wheel_link">
+    <link name="right_wheel_link">
         <visual>
             <origin xyz="0 0 0" rpy="1.57 0 0"/>
@@ -46,5 +46,5 @@
             <origin xyz="0 0 0" rpy="1.57 0 0"/>
             <geometry>
-                <mesh filename="package://amr_project/meshes/wheel_right_link.STL"/>
+                <cylinder radius="0.033" length="0.018"/>
             </geometry>
         </collision>
@@ -52,6 +52,6 @@
             <origin xyz="0 0 0" rpy="0 0 0"/>
             <mass value="0.5"/>
-            <inertia ixx="0.005" ixy="0.0" ixz="0.0"
-                     iyy="0.005" iyz="0.0" izz="0.005"/>
+            <inertia ixx="0.000354" ixy="0.0" ixz="0.0"
+                     iyy="0.000354" iyz="0.0" izz="0.000544"/>
         </inertial>
     </link>
@@ -75,5 +75,5 @@
             <origin xyz="0 0 0" rpy="-1.57 0 0"/>
             <geometry>
-                <mesh filename="package://amr_project/meshes/wheel_left_link.STL"/>
+                <cylinder radius="0.033" length="0.018"/>
             </geometry>
         </collision>
@@ -81,6 +81,6 @@
             <origin xyz="0 0 0" rpy="0 0 0"/>
             <mass value="0.5"/>
-            <inertia ixx="0.005" ixy="0.0" ixz="0.0"
-                     iyy="0.005" iyz="0.0" izz="0.005"/>
+            <inertia ixx="0.000354" ixy="0.0" ixz="0.0"
+                     iyy="0.000354" iyz="0.0" izz="0.000544"/>
         </inertial>
     </link>
@@ -104,12 +104,12 @@
             <origin xyz="0 0 0" rpy="0 0 0"/>
             <geometry>
-                <mesh filename="package://amr_project/meshes/caster_front_link.STL"/>
-            </geometry>
-        </collision>
-        <inertial>
-            <origin xyz="0 0 0" rpy="0 0 0"/>
-            <mass value="0.2"/>
-            <inertia ixx="0.002" ixy="0.0" ixz="0.0"
-                     iyy="0.002" iyz="0.0" izz="0.002"/>
+                <sphere radius="0.005"/>
+            </geometry>
+        </collision>
+        <inertial>
+            <origin xyz="0 0 0" rpy="0 0 0"/>
+            <mass value="0.1"/>
+            <inertia ixx="0.00001" ixy="0.0" ixz="0.0"
+                     iyy="0.00001" iyz="0.0" izz="0.00001"/>
         </inertial>
     </link>
@@ -132,12 +132,12 @@
             <origin xyz="0 0 0" rpy="0 0 0"/>
             <geometry>
-                <mesh filename="package://amr_project/meshes/caster_rear_link.STL"/>
-            </geometry>
-        </collision>
-        <inertial>
-            <origin xyz="0 0 0" rpy="0 0 0"/>
-            <mass value="0.2"/>
-            <inertia ixx="0.002" ixy="0.0" ixz="0.0"
-                     iyy="0.002" iyz="0.0" izz="0.002"/>
+                <sphere radius="0.005"/>
+            </geometry>
+        </collision>
+        <inertial>
+            <origin xyz="0 0 0" rpy="0 0 0"/>
+            <mass value="0.1"/>
+            <inertia ixx="0.00001" ixy="0.0" ixz="0.0"
+                     iyy="0.00001" iyz="0.0" izz="0.00001"/>
         </inertial>
     </link>
@@ -147,3 +147,59 @@
         <origin xyz="-0.04755 0 -0.0275" rpy="0 0 0"/>
     </joint>
+    <link name="imu_link">
+        <visual>
+            <origin xyz="0 0 0" rpy="0 0 0"/>
+            <geometry>
+                <mesh filename="package://amr_project/meshes/imu_link.STL"/>
+            </geometry>
+            <material name="imulink">
+                <color rgba="1 1 0 1"/>
+            </material>
+        </visual>
+        <collision>
+            <origin xyz="0 0 0" rpy="0 0 0"/>
+            <geometry>
+                <box size="0.02 0.02 0.01"/>
+            </geometry>
+        </collision>
+        <inertial>
+            <origin xyz="0 0 0" rpy="0 0 0"/>
+            <mass value="0.05"/>
+            <inertia ixx="0.00001" ixy="0.0" ixz="0.0"
+                     iyy="0.00001" iyz="0.0" izz="0.00001"/>
+        </inertial>
+    </link>
+    <joint name="imu_joint" type="fixed">
+        <parent link="base_link"/>
+        <child link="imu_link"/>
+        <origin xyz="0 0 0.03" rpy="0 0 0"/>
+    </joint>
+    <link name="laser_link">
+        <visual>
+            <origin xyz="0 0 0" rpy="0 0 0"/>
+            <geometry>
+                <mesh filename="package://amr_project/meshes/laser_link.STL"/>
+            </geometry>
+            <material name="laserlink">
+                <color rgba="1 0 1 1"/>
+            </material>
+        </visual>
+        <collision>
+            <origin xyz="0 0 0" rpy="0 0 0"/>
+            <geometry>
+                <cylinder radius="0.025" length="0.03"/>
+            </geometry>
+        </collision>
+        <inertial>
+            <origin xyz="0 0 0" rpy="0 0 0"/>
+            <mass value="0.2"/>
+            <inertia ixx="0.0001" ixy="0.0" ixz="0.0"
+                     iyy="0.0001" iyz="0.0" izz="0.0001"/>
+        </inertial>
+    </link>
+    <joint name="laser_joint" type="fixed">
+        <parent link="base_link"/>
+        <child link="laser_link"/>
+        <origin xyz="0.05 0 0.05" rpy="0 0 0"/>
+    </joint>
 </robot>

File: src/amr_project/robot_description/urdf/bot_gazebo.xacro (robot description, xacro)
@@ -1,5 +1,4 @@
 <?xml version="1.0"?>
 <robot xmlns:xacro="http://www.ros.org/wiki/xacro" name="bot_gazebo">
-    <!-- Gazebo properties for right wheel -->
     <gazebo reference="right_wheel_link">
         <mu1>1.0</mu1>
@@ -16,5 +15,4 @@
         </material>
     </gazebo>
-    <!-- Gazebo properties for left wheel -->
     <gazebo reference="left_wheel_link">
         <mu1>1.0</mu1>
@@ -31,5 +29,4 @@
         </material>
     </gazebo>
-    <!-- Gazebo properties for front caster -->
     <gazebo reference="caster_front_link">
         <mu1>0.01</mu1>
@@ -44,5 +41,4 @@
         </material>
     </gazebo>
-    <!-- Gazebo properties for rear caster -->
     <gazebo reference="caster_rear_link">
         <mu1>0.01</mu1>
@@ -57,5 +53,4 @@
         </material>
     </gazebo>
-    <!-- Make base_link visible -->
     <gazebo reference="base_link">
         <material>
@@ -65,36 +60,95 @@
         </material>
     </gazebo>
-    <!-- ros2_control configuration -->
-    <ros2_control name="GazeboSystem" type="system">
-        <hardware>
-            <plugin>gz_ros2_control/GazeboSimSystem</plugin>
-        </hardware>
-        <!-- Right wheel joint -->
-        <joint name="right_wheel_joint">
-            <command_interface name="velocity">
-                <param name="min">-10</param>
-                <param name="max">10</param>
-            </command_interface>
-            <state_interface name="position"/>
-            <state_interface name="velocity"/>
-            <state_interface name="effort"/>
-        </joint>
-        <!-- Left wheel joint -->
-        <joint name="left_wheel_joint">
-            <command_interface name="velocity">
-                <param name="min">-10</param>
-                <param name="max">10</param>
-            </command_interface>
-            <state_interface name="position"/>
-            <state_interface name="velocity"/>
-            <state_interface name="effort"/>
-        </joint>
-    </ros2_control>
-    <!-- Gazebo ros2_control plugin -->
-    <gazebo>
-        <plugin filename="gz_ros2_control-system"
-                name="gz_ros2_control::GazeboSimROS2ControlPlugin">
-            <parameters>$(find bot_controller)/config/controller.yaml</parameters>
-        </plugin>
+    <gazebo reference="imu_link">
+        <material>
+            <ambient>1.0 1.0 0.0 1</ambient>
+            <diffuse>1.0 1.0 0.0 1</diffuse>
+        </material>
+    </gazebo>
+    <gazebo reference="laser_link">
+        <material>
+            <ambient>1.0 0.0 1.0 1</ambient>
+            <diffuse>1.0 0.0 1.0 1</diffuse>
+        </material>
+    </gazebo>
+    <gazebo reference="imu_link">
+        <sensor name="imu_sensor" type="imu">
+            <always_on>true</always_on>
+            <update_rate>100</update_rate>
+            <visualize>true</visualize>
+            <topic>imu</topic>
+            <enable_metrics>true</enable_metrics>
+            <imu>
+                <angular_velocity>
+                    <x>
+                        <noise type="gaussian">
+                            <mean>0.0</mean>
+                            <stddev>2e-4</stddev>
+                        </noise>
+                    </x>
+                    <y>
+                        <noise type="gaussian">
+                            <mean>0.0</mean>
+                            <stddev>2e-4</stddev>
+                        </noise>
+                    </y>
+                    <z>
+                        <noise type="gaussian">
+                            <mean>0.0</mean>
+                            <stddev>2e-4</stddev>
+                        </noise>
+                    </z>
+                </angular_velocity>
+                <linear_acceleration>
+                    <x>
+                        <noise type="gaussian">
+                            <mean>0.0</mean>
+                            <stddev>1.7e-2</stddev>
+                        </noise>
+                    </x>
+                    <y>
+                        <noise type="gaussian">
+                            <mean>0.0</mean>
+                            <stddev>1.7e-2</stddev>
+                        </noise>
+                    </y>
+                    <z>
+                        <noise type="gaussian">
+                            <mean>0.0</mean>
+                            <stddev>1.7e-2</stddev>
+                        </noise>
+                    </z>
+                </linear_acceleration>
+            </imu>
+        </sensor>
+    </gazebo>
+    <gazebo reference="laser_link">
+        <sensor name="laser_sensor" type="gpu_lidar">
+            <always_on>true</always_on>
+            <update_rate>10</update_rate>
+            <visualize>true</visualize>
+            <topic>scan</topic>
+            <enable_metrics>true</enable_metrics>
+            <lidar>
+                <scan>
+                    <horizontal>
+                        <samples>360</samples>
+                        <resolution>1</resolution>
+                        <min_angle>-3.14159</min_angle>
+                        <max_angle>3.14159</max_angle>
+                    </horizontal>
+                </scan>
+                <range>
+                    <min>0.12</min>
+                    <max>10.0</max>
+                    <resolution>0.01</resolution>
+                </range>
+                <noise>
+                    <type>gaussian</type>
+                    <mean>0.0</mean>
+                    <stddev>0.01</stddev>
+                </noise>
+            </lidar>
+        </sensor>
     </gazebo>
 </robot>

Commit message: edited the urdf file for placing the laser on right position

File: src/amr_project/robot_description/urdf/bot.urdf.xacro (robot description, xacro)
@@ -177,5 +177,5 @@
     <link name="laser_link">
         <visual>
-            <origin xyz="0 0 0" rpy="0 0 0"/>
+            <origin xyz="-0.0050526 -0.0023221 0.1208" rpy="0 0 3.14"/>
             <geometry>
                 <mesh filename="package://amr_project/meshes/laser_link.STL"/>
