Commit message: updated the urdf file for stereo camera setup

File: src/amr_project/robot_description/urdf/bot.urdf.xacro (robot description, xacro)
@@ -3,27 +3,40 @@
     <xacro:arg name="is_ignition" default="true"/>
     <xacro:include filename="$(find amr_project)/urdf/bot_gazebo.xacro"/>
-    <xacro:include filename="$(find amr_project)/urdf/amr_controller.xacro"/>
+    <xacro:include filename="$(find amr_project)/urdf/bot_ros2_control.xacro"/>
+    <material name="blue">
+        <color rgba="0 0 0.8 1"/>
+    </material>
+    <material name="red">
+        <color rgba="0.8 0 0 1"/>
+    </material>
+    <material name="green">
+        <color rgba="0 0.8 0 1"/>
+    </material>
+    <material name="black">
+        <color rgba="0.15 0.15 0.15 1"/>
+    </material>
+    <material name="white">
+        <color rgba="0.9 0.9 0.9 1"/>
+    </material>
     <link name="base_footprint"/>
     <link name="base_link">
         <visual>
-            <origin xyz="0 0 0" rpy="0 0 0"/>
-            <geometry>
-                <mesh filename="package://amr_project/meshes/base_link.STL"/>
-            </geometry>
-            <material name="baselink">
-                <color rgba="0 0 1 1"/>
-            </material>
-        </visual>
-        <collision>
-            <origin xyz="0 0 0" rpy="0 0 0"/>
-            <geometry>
-                <mesh filename="package://amr_project/meshes/base_link.STL"/>
-            </geometry>
-        </collision>
-        <inertial>
-            <origin xyz="0 0 0" rpy="0 0 0"/>
-            <mass value="5.0"/>
-            <inertia ixx="0.0347" ixy="0.0" ixz="0.0"
-                     iyy="0.0347" iyz="0.0" izz="0.0625"/>
+            <origin xyz="0 0 0.015" rpy="0 0 0"/>
+            <geometry>
+                <box size="0.15 0.12 0.03"/>
+            </geometry>
+            <material name="blue"/>
+        </visual>
+        <collision>
+            <origin xyz="0 0 0.015" rpy="0 0 0"/>
+            <geometry>
+                <box size="0.15 0.12 0.03"/>
+            </geometry>
+        </collision>
+        <inertial>
+            <origin xyz="0 0 0.015" rpy="0 0 0"/>
+            <mass value="2.0"/>
+            <inertia ixx="0.0067" ixy="0.0" ixz="0.0"
+                     iyy="0.0100" iyz="0.0" izz="0.0150"/>
         </inertial>
     </link>
@@ -35,23 +48,21 @@
     <link name="right_wheel_link">
         <visual>
-            <origin xyz="0 0 0" rpy="1.57 0 0"/>
-            <geometry>
-                <mesh filename="package://amr_project/meshes/wheel_right_link.STL"/>
-            </geometry>
-            <material name="rwlink">
-                <color rgba="1 0 0 1"/>
-            </material>
-        </visual>
-        <collision>
-            <origin xyz="0 0 0" rpy="1.57 0 0"/>
-            <geometry>
-                <cylinder radius="0.033" length="0.018"/>
-            </geometry>
-        </collision>
-        <inertial>
-            <origin xyz="0 0 0" rpy="0 0 0"/>
-            <mass value="0.5"/>
-            <inertia ixx="0.000354" ixy="0.0" ixz="0.0"
-                     iyy="0.000354" iyz="0.0" izz="0.000544"/>
+            <origin xyz="0 0 0" rpy="1.5707963 0 0"/>
+            <geometry>
+                <cylinder radius="0.033" length="0.02"/>
+            </geometry>
+            <material name="black"/>
+        </visual>
+        <collision>
+            <origin xyz="0 0 0" rpy="1.5707963 0 0"/>
+            <geometry>
+                <cylinder radius="0.033" length="0.02"/>
+            </geometry>
+        </collision>
+        <inertial>
+            <origin xyz="0 0 0" rpy="0 0 0"/>
+            <mass value="0.2"/>
+            <inertia ixx="0.000139" ixy="0.0" ixz="0.0"
+                     iyy="0.000139" iyz="0.0" izz="0.000217"/>
         </inertial>
     </link>
@@ -64,23 +75,21 @@
     <link name="left_wheel_link">
         <visual>
-            <origin xyz="0 0 0" rpy="-1.57 0 0"/>
-            <geometry>
-                <mesh filename="package://amr_project/meshes/wheel_left_link.STL"/>
-            </geometry>
-            <material name="lwlink">
-                <color rgba="1 0 0 1"/>
-            </material>
-        </visual>
-        <collision>
-            <origin xyz="0 0 0" rpy="-1.57 0 0"/>
-            <geometry>
-                <cylinder radius="0.033" length="0.018"/>
-            </geometry>
-        </collision>
-        <inertial>
-            <origin xyz="0 0 0" rpy="0 0 0"/>
-            <mass value="0.5"/>
-            <inertia ixx="0.000354" ixy="0.0" ixz="0.0"
-                     iyy="0.000354" iyz="0.0" izz="0.000544"/>
+            <origin xyz="0 0 0" rpy="-1.5707963 0 0"/>
+            <geometry>
+                <cylinder radius="0.033" length="0.02"/>
+            </geometry>
+            <material name="black"/>
+        </visual>
+        <collision>
+            <origin xyz="0 0 0" rpy="-1.5707963 0 0"/>
+            <geometry>
+                <cylinder radius="0.033" length="0.02"/>
+            </geometry>
+        </collision>
+        <inertial>
+            <origin xyz="0 0 0" rpy="0 0 0"/>
+            <mass value="0.2"/>
+            <inertia ixx="0.000139" ixy="0.0" ixz="0.0"
+                     iyy="0.000139" iyz="0.0" izz="0.000217"/>
         </inertial>
     </link>
@@ -95,14 +104,90 @@
             <origin xyz="0 0 0" rpy="0 0 0"/>
             <geometry>
-                <mesh filename="package://amr_project/meshes/caster_front_link.STL"/>
-            </geometry>
-            <material name="cflink">
-                <color rgba="0 1 0 1"/>
-            </material>
-        </visual>
-        <collision>
-            <origin xyz="0 0 0" rpy="0 0 0"/>
-            <geometry>
-                <sphere radius="0.005"/>
+                <sphere radius="0.008"/>
+            </geometry>
+            <material name="white"/>
+        </visual>
+        <collision>
+            <origin xyz="0 0 0" rpy="0 0 0"/>
+            <geometry>
+                <sphere radius="0.008"/>
+            </geometry>
+        </collision>
+        <inertial>
+            <origin xyz="0 0 0" rpy="0 0 0"/>
+            <mass value="0.05"/>
+            <inertia ixx="0.000001" ixy="0.0" ixz="0.0"
+                     iyy="0.000001" iyz="0.0" izz="0.000001"/>
+        </inertial>
+    </link>
+    <joint name="caster_front_joint" type="fixed">
+        <parent link="base_link"/>
+        <child link="caster_front_link"/>
+        <origin xyz="0.05 0 -0.025" rpy="0 0 0"/>
+    </joint>
+    <link name="caster_rear_link">
+        <visual>
+            <origin xyz="0 0 0" rpy="0 0 0"/>
+            <geometry>
+                <sphere radius="0.008"/>
+            </geometry>
+            <material name="white"/>
+        </visual>
+        <collision>
+            <origin xyz="0 0 0" rpy="0 0 0"/>
+            <geometry>
+                <sphere radius="0.008"/>
+            </geometry>
+        </collision>
+        <inertial>
+            <origin xyz="0 0 0" rpy="0 0 0"/>
+            <mass value="0.05"/>
+            <inertia ixx="0.000001" ixy="0.0" ixz="0.0"
+                     iyy="0.000001" iyz="0.0" izz="0.000001"/>
+        </inertial>
+    </link>
+    <joint name="caster_rear_joint" type="fixed">
+        <parent link="base_link"/>
+        <child link="caster_rear_link"/>
+        <origin xyz="-0.05 0 -0.025" rpy="0 0 0"/>
+    </joint>
+    <link name="imu_link">
+        <visual>
+            <origin xyz="0 0 0" rpy="0 0 0"/>
+            <geometry>
+                <box size="0.02 0.02 0.01"/>
+            </geometry>
+            <material name="red"/>
+        </visual>
+        <collision>
+            <origin xyz="0 0 0" rpy="0 0 0"/>
+            <geometry>
+                <box size="0.02 0.02 0.01"/>
+            </geometry>
+        </collision>
+        <inertial>
+            <origin xyz="0 0 0" rpy="0 0 0"/>
+            <mass value="0.02"/>
+            <inertia ixx="0.000001" ixy="0.0" ixz="0.0"
+                     iyy="0.000001" iyz="0.0" izz="0.000001"/>
+        </inertial>
+    </link>
+    <joint name="imu_joint" type="fixed">
+        <parent link="base_link"/>
+        <child link="imu_link"/>
+        <origin xyz="0 0 0.035" rpy="0 0 0"/>
+    </joint>
+    <link name="laser_link">
+        <visual>
+            <origin xyz="0 0 0" rpy="0 0 0"/>
+            <geometry>
+                <cylinder radius="0.025" length="0.03"/>
+            </geometry>
+            <material name="red"/>
+        </visual>
+        <collision>
+            <origin xyz="0 0 0" rpy="0 0 0"/>
+            <geometry>
+                <cylinder radius="0.025" length="0.03"/>
             </geometry>
         </collision>
@@ -114,51 +199,21 @@
         </inertial>
     </link>
-    <joint name="caster_front_joint" type="fixed">
-        <parent link="base_link"/>
-        <child link="caster_front_link"/>
-        <origin xyz="0.04755 0 -0.0275" rpy="0 0 0"/>
-    </joint>
-    <link name="caster_rear_link">
-        <visual>
-            <origin xyz="0 0 0" rpy="0 0 0"/>
-            <geometry>
-                <mesh filename="package://amr_project/meshes/caster_rear_link.STL"/>
-            </geometry>
-            <material name="crlink">
-                <color rgba="0 1 0 1"/>
-            </material>
-        </visual>
-        <collision>
-            <origin xyz="0 0 0" rpy="0 0 0"/>
-            <geometry>
-                <sphere radius="0.005"/>
-            </geometry>
-        </collision>
-        <inertial>
-            <origin xyz="0 0 0" rpy="0 0 0"/>
-            <mass value="0.1"/>
-            <inertia ixx="0.00001" ixy="0.0" ixz="0.0"
-                     iyy="0.00001" iyz="0.0" izz="0.00001"/>
-        </inertial>
-    </link>
-    <joint name="caster_rear_joint" type="fixed">
-        <parent link="base_link"/>
-        <child link="caster_rear_link"/>
-        <origin xyz="-0.04755 0 -0.0275" rpy="0 0 0"/>
-    </joint>
-    <link name="imu_link">
-        <visual>
-            <origin xyz="0 0 0" rpy="0 0 0"/>
-            <geometry>
-                <mesh filename="package://amr_project/meshes/imu_link.STL"/>
-            </geometry>
-            <material name="imulink">
-                <color rgba="1 1 0 1"/>
-            </material>
-        </visual>
-        <collision>
-            <origin xyz="0 0 0" rpy="0 0 0"/>
-            <geometry>
-                <box size="0.02 0.02 0.01"/>
+    <joint name="laser_joint" type="fixed">
+        <parent link="base_link"/>
+        <child link="laser_link"/>
+        <origin xyz="0.05 0 0.05" rpy="0 0 0"/>
+    </joint>
+    <link name="camera_mount_link">
+        <visual>
+            <origin xyz="0 0 0" rpy="0 0 0"/>
+            <geometry>
+                <box size="0.02 0.10 0.015"/>
+            </geometry>
+            <material name="black"/>
+        </visual>
+        <collision>
+            <origin xyz="0 0 0" rpy="0 0 0"/>
+            <geometry>
+                <box size="0.02 0.10 0.015"/>
             </geometry>
         </collision>
@@ -170,36 +225,104 @@
         </inertial>
     </link>
-    <joint name="imu_joint" type="fixed">
-        <parent link="base_link"/>
-        <child link="imu_link"/>
-        <origin xyz="0 0 0.03" rpy="0 0 0"/>
-    </joint>
-    <link name="laser_link">
-        <visual>
-            <origin xyz="-0.0050526 -0.0023221 0.1208" rpy="0 0 3.14"/>
-            <geometry>
-                <mesh filename="package://amr_project/meshes/laser_link.STL"/>
-            </geometry>
-            <material name="laserlink">
-                <color rgba="1 0 1 1"/>
-            </material>
-        </visual>
-        <collision>
-            <origin xyz="0 0 0" rpy="0 0 0"/>
-            <geometry>
-                <cylinder radius="0.025" length="0.03"/>
-            </geometry>
-        </collision>
-        <inertial>
-            <origin xyz="0 0 0" rpy="0 0 0"/>
-            <mass value="0.2"/>
-            <inertia ixx="0.0001" ixy="0.0" ixz="0.0"
-                     iyy="0.0001" iyz="0.0" izz="0.0001"/>
-        </inertial>
-    </link>
-    <joint name="laser_joint" type="fixed">
-        <parent link="base_link"/>
-        <child link="laser_link"/>
-        <origin xyz="0.05 0 0.05" rpy="0 0 0"/>
+    <joint name="camera_mount_joint" type="fixed">
+        <parent link="base_link"/>
+        <child link="camera_mount_link"/>
+        <origin xyz="0.065 0 0.07" rpy="0 0 0"/>
+    </joint>
+    <link name="camera_left_link">
+        <visual>
+            <origin xyz="0 0 0" rpy="0 0 0"/>
+            <geometry>
+                <box size="0.01 0.025 0.025"/>
+            </geometry>
+            <material name="black"/>
+        </visual>
+        <collision>
+            <origin xyz="0 0 0" rpy="0 0 0"/>
+            <geometry>
+                <box size="0.01 0.025 0.025"/>
+            </geometry>
+        </collision>
+        <inertial>
+            <origin xyz="0 0 0" rpy="0 0 0"/>
+            <mass value="0.03"/>
+            <inertia ixx="0.000001" ixy="0.0" ixz="0.0"
+                     iyy="0.000001" iyz="0.0" izz="0.000001"/>
+        </inertial>
+    </link>
+    <joint name="camera_left_joint" type="fixed">
+        <parent link="camera_mount_link"/>
+        <child link="camera_left_link"/>
+        <origin xyz="0 0.0375 0" rpy="0 0 0"/>
+    </joint>
+    <link name="camera_left_optical_frame"/>
+    <joint name="camera_left_optical_joint" type="fixed">
+        <parent link="camera_left_link"/>
+        <child link="camera_left_optical_frame"/>
+        <origin xyz="0 0 0" rpy="-1.5707963 0 -1.5707963"/>
+    </joint>
+    <link name="camera_right_link">
+        <visual>
+            <origin xyz="0 0 0" rpy="0 0 0"/>
+            <geometry>
+                <box size="0.01 0.025 0.025"/>
+            </geometry>
+            <material name="black"/>
+        </visual>
+        <collision>
+            <origin xyz="0 0 0" rpy="0 0 0"/>
+            <geometry>
+                <box size="0.01 0.025 0.025"/>
+            </geometry>
+        </collision>
+        <inertial>
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