Commit message: did all the final changes and now robot is ready to map

File: src/amr_project/robot_description/urdf/bot.urdf.xacro (robot description, xacro)
@@ -116,7 +116,7 @@
         <inertial>
             <origin xyz="0 0 0" rpy="0 0 0"/>
-            <mass value="0.05"/>
-            <inertia ixx="0.000001" ixy="0.0" ixz="0.0"
-                     iyy="0.000001" iyz="0.0" izz="0.000001"/>
+            <mass value="0.2"/>
+            <inertia ixx="0.001" ixy="0.0" ixz="0.0"
+                     iyy="0.001" iyz="0.0" izz="0.001"/>
         </inertial>
     </link>
@@ -142,7 +142,7 @@
         <inertial>
             <origin xyz="0 0 0" rpy="0 0 0"/>
-            <mass value="0.05"/>
-            <inertia ixx="0.000001" ixy="0.0" ixz="0.0"
-                     iyy="0.000001" iyz="0.0" izz="0.000001"/>
+            <mass value="0.2"/>
+            <inertia ixx="0.001" ixy="0.0" ixz="0.0"
+                     iyy="0.001" iyz="0.0" izz="0.001"/>
         </inertial>
     </link>
@@ -169,6 +169,6 @@
             <origin xyz="0 0 0" rpy="0 0 0"/>
             <mass value="0.02"/>
-            <inertia ixx="0.000001" ixy="0.0" ixz="0.0"
-                     iyy="0.000001" iyz="0.0" izz="0.000001"/>
+            <inertia ixx="0.001" ixy="0.0" ixz="0.0"
+                     iyy="0.001" iyz="0.0" izz="0.001"/>
         </inertial>
     </link>
@@ -194,7 +194,7 @@
         <inertial>
             <origin xyz="0 0 0" rpy="0 0 0"/>
-            <mass value="0.1"/>
-            <inertia ixx="0.00001" ixy="0.0" ixz="0.0"
-                     iyy="0.00001" iyz="0.0" izz="0.00001"/>
+            <mass value="0.2"/>
+            <inertia ixx="0.001" ixy="0.0" ixz="0.0"
+                     iyy="0.001" iyz="0.0" izz="0.001"/>
         </inertial>
     </link>
@@ -221,6 +221,6 @@
             <origin xyz="0 0 0" rpy="0 0 0"/>
             <mass value="0.05"/>
-            <inertia ixx="0.00001" ixy="0.0" ixz="0.0"
-                     iyy="0.00001" iyz="0.0" izz="0.00001"/>
+            <inertia ixx="0.001" ixy="0.0" ixz="0.0"
+                     iyy="0.001" iyz="0.0" izz="0.001"/>
         </inertial>
     </link>
@@ -246,7 +246,7 @@
         <inertial>
             <origin xyz="0 0 0" rpy="0 0 0"/>
-            <mass value="0.03"/>
-            <inertia ixx="0.000001" ixy="0.0" ixz="0.0"
-                     iyy="0.000001" iyz="0.0" izz="0.000001"/>
+            <mass value="0.2"/>
+            <inertia ixx="0.001" ixy="0.0" ixz="0.0"
+                     iyy="0.001" iyz="0.0" izz="0.001"/>
         </inertial>
     </link>
@@ -278,7 +278,7 @@
         <inertial>
             <origin xyz="0 0 0" rpy="0 0 0"/>
-            <mass value="0.03"/>
-            <inertia ixx="0.000001" ixy="0.0" ixz="0.0"
-                     iyy="0.000001" iyz="0.0" izz="0.000001"/>
+            <mass value="0.2"/>
+            <inertia ixx="0.001" ixy="0.0" ixz="0.0"
+                     iyy="0.001" iyz="0.0" izz="0.001"/>
         </inertial>
     </link>
@@ -310,7 +310,7 @@
         <inertial>
             <origin xyz="0 0 0" rpy="0 0 0"/>
-            <mass value="0.03"/>
-            <inertia ixx="0.000001" ixy="0.0" ixz="0.0"
-                     iyy="0.000001" iyz="0.0" izz="0.000001"/>
+            <mass value="0.2"/>
+            <inertia ixx="0.001" ixy="0.0" ixz="0.0"
+                     iyy="0.001" iyz="0.0" izz="0.001"/>
         </inertial>
     </link>

File: src/amr_project/robot_description/urdf/bot_gazebo.xacro (robot description, xacro)
@@ -1,4 +1,20 @@
 <?xml version="1.0"?>
 <robot xmlns:xacro="http://www.ros.org/wiki/xacro" name="bot_gazebo">
+    <gazebo>
+        <plugin
+            filename="ignition-gazebo-diff-drive-system"
+            name="ignition::gazebo::systems::DiffDrive">
+            <left_joint>left_wheel_joint</left_joint>
+            <right_joint>right_wheel_joint</right_joint>
+            <wheel_separation>0.14</wheel_separation>
+            <wheel_radius>0.033</wheel_radius>
+            <topic>cmd_vel</topic>
+            <odom_topic>odom</odom_topic>
+            <tf_topic>tf</tf_topic>
+            <frame_id>odom</frame_id>
+            <child_frame_id>base_footprint</child_frame_id>
+            <odom_publish_frequency>30</odom_publish_frequency>
+        </plugin>
+    </gazebo>
     <gazebo reference="right_wheel_link">
         <mu1>1.0</mu1>
@@ -6,7 +22,4 @@
         <kp>1000000.0</kp>
         <kd>10.0</kd>
-        <minDepth>0.001</minDepth>
-        <maxVel>1.0</maxVel>
-        <fdir1>1 0 0</fdir1>
         <material>Gazebo/Black</material>
     </gazebo>
@@ -16,7 +29,4 @@
         <kp>1000000.0</kp>
         <kd>10.0</kd>
-        <minDepth>0.001</minDepth>
-        <maxVel>1.0</maxVel>
-        <fdir1>1 0 0</fdir1>
         <material>Gazebo/Black</material>
     </gazebo>
@@ -24,6 +34,4 @@
         <mu1>0.0</mu1>
         <mu2>0.0</mu2>
-        <kp>1000000.0</kp>
-        <kd>100.0</kd>
         <material>Gazebo/White</material>
     </gazebo>
@@ -31,19 +39,5 @@
         <mu1>0.0</mu1>
         <mu2>0.0</mu2>
-        <kp>1000000.0</kp>
-        <kd>100.0</kd>
         <material>Gazebo/White</material>
-    </gazebo>
-    <gazebo reference="base_link">
-        <material>Gazebo/Blue</material>
-    </gazebo>
-    <gazebo reference="imu_link">
-        <material>Gazebo/Red</material>
-    </gazebo>
-    <gazebo reference="laser_link">
-        <material>Gazebo/Red</material>
-    </gazebo>
-    <gazebo reference="camera_mount_link">
-        <material>Gazebo/Black</material>
     </gazebo>
     <gazebo reference="imu_link">
@@ -51,19 +45,9 @@
             <always_on>true</always_on>
             <update_rate>100</update_rate>
-            <visualize>false</visualize>
             <topic>imu</topic>
-            <imu>
-                <angular_velocity>
-                    <x><noise type="gaussian"><mean>0.0</mean><stddev>2e-4</stddev></noise></x>
-                    <y><noise type="gaussian"><mean>0.0</mean><stddev>2e-4</stddev></noise></y>
-                    <z><noise type="gaussian"><mean>0.0</mean><stddev>2e-4</stddev></noise></z>
-                </angular_velocity>
-                <linear_acceleration>
-                    <x><noise type="gaussian"><mean>0.0</mean><stddev>1.7e-2</stddev></noise></x>
-                    <y><noise type="gaussian"><mean>0.0</mean><stddev>1.7e-2</stddev></noise></y>
-                    <z><noise type="gaussian"><mean>0.0</mean><stddev>1.7e-2</stddev></noise></z>
-                </linear_acceleration>
-            </imu>
+            <gz_frame_id>imu_link</gz_frame_id>
+            <imu/>
         </sensor>
+        <material>Gazebo/Red</material>
     </gazebo>
     <gazebo reference="laser_link">
@@ -86,97 +70,11 @@
                     <min>0.12</min>
                     <max>10.0</max>
-                    <resolution>0.01</resolution>
                 </range>
-                <noise>
-                    <type>gaussian</type>
-                    <mean>0.0</mean>
-                    <stddev>0.01</stddev>
-                </noise>
             </lidar>
         </sensor>
+        <material>Gazebo/Red</material>
     </gazebo>
-    <gazebo reference="camera_left_link">
-        <sensor name="left_camera" type="camera">
-            <always_on>true</always_on>
-            <update_rate>30</update_rate>
-            <visualize>false</visualize>
-            <topic>camera/left</topic>
-            <camera>
-                <horizontal_fov>1.5708</horizontal_fov>
-                <image>
-                    <width>640</width>
-                    <height>480</height>
-                    <format>R8G8B8</format>
-                </image>
-                <clip>
-                    <near>0.05</near>
-                    <far>100</far>
-                </clip>
-                <noise>
-                    <type>gaussian</type>
-                    <mean>0.0</mean>
-                    <stddev>0.007</stddev>
-                </noise>
-            </camera>
-        </sensor>
-    </gazebo>
-    <gazebo reference="camera_right_link">
-        <sensor name="right_camera" type="camera">
-            <always_on>true</always_on>
-            <update_rate>30</update_rate>
-            <visualize>false</visualize>
-            <topic>camera/right</topic>
-            <camera>
-                <horizontal_fov>1.5708</horizontal_fov>
-                <image>
-                    <width>640</width>
-                    <height>480</height>
-                    <format>R8G8B8</format>
-                </image>
-                <clip>
-                    <near>0.05</near>
-                    <far>100</far>
-                </clip>
-                <noise>
-                    <type>gaussian</type>
-                    <mean>0.0</mean>
-                    <stddev>0.007</stddev>
-                </noise>
-            </camera>
-        </sensor>
-    </gazebo>
-    <gazebo reference="camera_center_link">
-        <sensor name="depth_camera" type="depth_camera">
-            <always_on>true</always_on>
-            <update_rate>30</update_rate>
-            <visualize>false</visualize>
-            <topic>camera/depth</topic>
-            <camera>
-                <horizontal_fov>1.5708</horizontal_fov>
-                <image>
-                    <width>640</width>
-                    <height>480</height>
-                    <format>R_FLOAT32</format>
-                </image>
-                <clip>
-                    <near>0.05</near>
-                    <far>10.0</far>
-                </clip>
-                <noise>
-                    <type>gaussian</type>
-                    <mean>0.0</mean>
-                    <stddev>0.01</stddev>
-                </noise>
-            </camera>
-        </sensor>
-    </gazebo>
-    <gazebo reference="laser_joint">
-        <preserveFixedJoint>true</preserveFixedJoint>
-    </gazebo>
-    <gazebo reference="imu_joint">
-        <preserveFixedJoint>true</preserveFixedJoint>
-    </gazebo>
-    <gazebo reference="camera_mount_joint">
-        <preserveFixedJoint>true</preserveFixedJoint>
-    </gazebo>
+    <gazebo reference="laser_joint"><preserveFixedJoint>true</preserveFixedJoint></gazebo>
+    <gazebo reference="imu_joint"><preserveFixedJoint>true</preserveFixedJoint></gazebo>
+    <gazebo reference="camera_mount_joint"><preserveFixedJoint>true</preserveFixedJoint></gazebo>
 </robot>
